File: SmoothieboardGlcdAdapter2.brd (EAGLE design)
At the start: 62.9 x 67.9 mm, 16 parts, among them IC1 7805TV

Commit message: recom outline
Routing:
- net GND: track 77.9 -> 81.8 mm
- net 5V: track 51.0 -> 49.9 mm
- net VBB: track 75.6 -> 75.2 mm, vias 2 -> 0
Changed lines of the file:
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@@
 <wire x1="108.9025" y1="44.1325" x2="110.1725" y2="44.1325" width="0.0508" layer="41"/>
 <text x="14.605" y="13.081" size="1.016" layer="121" ratio="16">5V</text>
-<text x="29.6545" y="35.687" size="1.016" layer="121" font="vector" ratio="10" rot="R270">P1.30</text>
-<text x="32.258" y="35.7505" size="1.016" layer="121" font="vector" ratio="10" rot="R270">P1.31</text>
-<text x="35.687" y="35.687" size="0.762" layer="121" font="vector" ratio="10" rot="R270">P1.23</text>
-<text x="38.227" y="35.56" size="0.762" layer="121" font="vector" ratio="10" rot="R270">P1.22</text>
-<text x="27.8765" y="35.814" size="0.8128" layer="121" font="vector" ratio="10" rot="R270">GND</text>
+<text x="29.6545" y="38.1" size="0.762" layer="121" font="vector" ratio="10" rot="R45">P1.30</text>
+<text x="32.1945" y="38.227" size="0.762" layer="121" font="vector" ratio="10" rot="R45">P1.31</text>
+<text x="34.671" y="38.1" size="0.762" layer="121" font="vector" ratio="10" rot="R45">P1.23</text>
+<text x="37.084" y="38.1" size="0.762" layer="121" font="vector" ratio="10" rot="R45">P1.22</text>
+<text x="27.2415" y="38.354" size="0.762" layer="121" font="vector" ratio="10" rot="R45">GND</text>
 <text x="43.1165" y="25.5905" size="1.016" layer="121" font="vector" ratio="10" rot="R90">P2.11</text>
 <text x="45.7835" y="25.5905" size="1.016" layer="121" font="vector" ratio="10" rot="R90">P3.26</text>
@@
 <wire x1="21.59" y1="59.69" x2="29.21" y2="59.69" width="0.4064" layer="22"/>
 <wire x1="29.21" y1="59.69" x2="29.21" y2="64.77" width="0.4064" layer="22"/>
-<wire x1="27.305" y1="29.972" x2="27.305" y2="23.749" width="0.254" layer="121"/>
-<wire x1="27.305" y1="23.749" x2="37.465" y2="23.749" width="0.254" layer="121"/>
-<wire x1="37.465" y1="23.749" x2="37.465" y2="29.972" width="0.254" layer="121"/>
 <wire x1="34.671" y1="37.846" x2="34.671" y2="36.449" width="0.3048" layer="22"/>
 <wire x1="65.913" y1="34.798" x2="73.279" y2="34.798" width="0.3048" layer="22"/>
@@
 <text x="47.0535" y="25.5905" size="1.016" layer="121" font="vector" ratio="10" rot="R90">ENC-B</text>
 <text x="49.5935" y="25.5905" size="1.016" layer="121" font="vector" ratio="10" rot="R90">ENC-A</text>
-<text x="30.861" y="35.6235" size="1.016" layer="121" font="vector" ratio="10" rot="R270">E-SW</text>
-<text x="33.401" y="35.6235" size="1.016" layer="121" font="vector" ratio="10" rot="R270">BUZZ</text>
+<text x="31.369" y="38.5445" size="0.762" layer="121" font="vector" ratio="10" rot="R45">E-SW</text>
+<text x="33.655" y="38.4175" size="0.762" layer="121" font="vector" ratio="10" rot="R45">BUZZ</text>
 <wire x1="21.463" y1="65.405" x2="52.705" y2="65.405" width="0.254" layer="20"/>
 <wire x1="52.705" y1="65.405" x2="53.975" y2="66.675" width="0.254" layer="20"/>
@@
 <wire x1="22.86" y1="30.48" x2="16.51" y2="24.13" width="0.254" layer="20"/>
 <text x="39.243" y="55.499" size="1.524" layer="121">version</text>
+<wire x1="27.305" y1="27.051" x2="27.305" y2="34.036" width="0.4064" layer="121"/>
+<wire x1="27.305" y1="34.036" x2="37.465" y2="34.036" width="0.4064" layer="121"/>
+<wire x1="37.465" y1="34.036" x2="37.465" y2="27.051" width="0.4064" layer="121"/>
+<wire x1="37.465" y1="27.051" x2="27.305" y2="27.051" width="0.4064" layer="121"/>
 </plain>
 <attributes>
@@
 <contactref element="EXP2" pad="2"/>
 <wire x1="50.546" y1="52.07" x2="56.134" y2="57.658" width="0.8128" layer="1"/>
-<wire x1="56.134" y1="57.658" x2="56.515" y2="57.658" width="0.8128" layer="1"/>
-<wire x1="56.515" y1="57.658" x2="59.817" y2="57.658" width="0.8128" layer="1"/>
+<wire x1="56.134" y1="57.658" x2="59.817" y2="57.658" width="0.8128" layer="1"/>
 <wire x1="59.817" y1="57.658" x2="61.5589" y2="55.9161" width="0.8128" layer="1"/>
 <wire x1="61.5589" y1="55.9161" x2="62.130396875" y2="55.9161" width="0.8128" layer="1"/>
@@
 <wire x1="28.194" y1="37.211" x2="28.2575" y2="37.1475" width="0.8128" layer="1"/>
 <contactref element="IC1" pad="2"/>
-<wire x1="28.2575" y1="37.1475" x2="28.2575" y2="35.4965" width="0.8128" layer="16"/>
-<wire x1="28.2575" y1="35.4965" x2="32.385" y2="31.369" width="0.8128" layer="16"/>
-<wire x1="32.385" y1="31.369" x2="32.385" y2="28.829" width="0.8128" layer="16"/>
-<wire x1="56.3245" y1="70.358" x2="56.515" y2="70.358" width="0.8128" layer="1"/>
-<wire x1="56.515" y1="70.358" x2="56.515" y2="57.658" width="0.8128" layer="1"/>
+<wire x1="56.515" y1="70.358" x2="56.515" y2="61.531496875" width="0.8128" layer="16"/>
+<wire x1="56.515" y1="61.531496875" x2="62.130396875" y2="55.9161" width="0.8128" layer="16"/>
+<wire x1="56.515" y1="70.358" x2="56.3245" y2="70.358" width="0" layer="19" extent="16-16"/>
+<wire x1="28.2575" y1="37.1475" x2="28.2575" y2="35.6235" width="0.8128" layer="1"/>
+<wire x1="28.2575" y1="35.6235" x2="32.385" y2="31.496" width="0.8128" layer="1"/>
+<wire x1="32.385" y1="31.496" x2="32.385" y2="28.829" width="0.8128" layer="1"/>
 </signal>
 <signal name="SD_MOSI">
@@
 <contactref element="JP17" pad="1"/>
 <contactref element="IC1" pad="1"/>
-<wire x1="58.293" y1="75.438" x2="59.182" y2="74.549" width="0.8128" layer="16"/>
-<wire x1="59.182" y1="74.549" x2="59.182" y2="62.738" width="0.8128" layer="16"/>
-<wire x1="59.182" y1="62.738" x2="47.752" y2="51.308" width="0.8128" layer="16"/>
-<wire x1="47.752" y1="51.308" x2="41.529" y2="51.308" width="0.8128" layer="16"/>
-<via x="41.529" y="51.308" extent="1-16" drill="0.6" diameter="1.016"/>
-<wire x1="41.529" y1="51.308" x2="31.877" y2="51.308" width="0.8128" layer="1"/>
-<via x="31.877" y="51.308" extent="1-16" drill="0.6" diameter="1.016"/>
-<wire x1="31.877" y1="51.308" x2="29.591" y2="51.308" width="0.8128" layer="16"/>
-<wire x1="29.591" y1="51.308" x2="25.146" y2="46.863" width="0.8128" layer="16"/>
-<wire x1="25.146" y1="46.863" x2="25.146" y2="34.544" width="0.8128" layer="16"/>
-<wire x1="25.146" y1="34.544" x2="29.845" y2="29.845" width="0.8128" layer="16"/>
-<wire x1="29.845" y1="29.845" x2="29.845" y2="28.829" width="0.8128" layer="16"/>
-<wire x1="56.3245" y1="75.438" x2="58.293" y2="75.438" width="0.8128" layer="16"/>
+<wire x1="56.3245" y1="75.438" x2="57.785" y2="75.438" width="0.8128" layer="1"/>
+<wire x1="57.785" y1="75.438" x2="59.182" y2="74.041" width="0.8128" layer="1"/>
+<wire x1="59.182" y1="74.041" x2="59.182" y2="65.913" width="0.8128" layer="1"/>
+<wire x1="59.182" y1="65.913" x2="45.339" y2="52.07" width="0.8128" layer="1"/>
+<wire x1="45.339" y1="52.07" x2="30.099" y2="52.07" width="0.8128" layer="1"/>
+<wire x1="30.099" y1="52.07" x2="25.4" y2="47.371" width="0.8128" layer="1"/>
+<wire x1="25.4" y1="47.371" x2="25.4" y2="30.226" width="0.8128" layer="1"/>
+<wire x1="25.4" y1="30.226" x2="26.797" y2="28.829" width="0.8128" layer="1"/>
+<wire x1="26.797" y1="28.829" x2="29.845" y2="28.829" width="0.8128" layer="1"/>
 </signal>
 <signal name="N$52">
@@
 <contactref element="D1" pad="C"/>
 <contactref element="EXP1" pad="1"/>
-<wire x1="52.451" y1="43.688" x2="52.451" y2="36.068" width="0.8128" layer="1"/>
-<wire x1="52.451" y1="36.068" x2="49.022" y2="32.639" width="0.8128" layer="1"/>
-<wire x1="49.022" y1="32.639" x2="34.925" y2="32.639" width="0.8128" layer="1"/>
-<wire x1="34.925" y1="32.639" x2="26.924" y2="32.639" width="0.8128" layer="1"/>
 <contactref element="IC1" pad="3"/>
-<wire x1="34.925" y1="28.829" x2="34.925" y2="32.639" width="0.8128" layer="1"/>
-<wire x1="26.924" y1="32.639" x2="25.4" y2="31.115" width="0.8128" layer="1"/>
-<wire x1="25.4" y1="31.115" x2="25.4" y2="28.575" width="0.8128" layer="1"/>
-<wire x1="25.4" y1="28.575" x2="19.812" y2="22.987" width="0.8128" layer="1"/>
+<wire x1="19.812" y1="22.987" x2="33.02" y2="22.987" width="0.8128" layer="1"/>
+<wire x1="33.02" y1="22.987" x2="34.798" y2="24.765" width="0.8128" layer="1"/>
+<wire x1="34.798" y1="24.765" x2="34.798" y2="28.702" width="0.8128" layer="1"/>
+<wire x1="34.798" y1="28.702" x2="34.925" y2="28.829" width="0.8128" layer="1"/>
+<wire x1="34.925" y1="28.829" x2="34.925" y2="30.734" width="0.8128" layer="1"/>
+<wire x1="34.925" y1="30.734" x2="36.576" y2="32.385" width="0.8128" layer="1"/>
+<wire x1="36.576" y1="32.385" x2="48.387" y2="32.385" width="0.8128" layer="1"/>
+<wire x1="48.387" y1="32.385" x2="53.721" y2="37.719" width="0.8128" layer="1"/>
+<wire x1="53.721" y1="37.719" x2="53.721" y2="41.275" width="0.8128" layer="1"/>
+<wire x1="53.721" y1="41.275" x2="52.578" y2="42.418" width="0.8128" layer="1"/>
+<wire x1="52.578" y1="42.418" x2="52.578" y2="43.561" width="0.8128" layer="1"/>
+<wire x1="52.578" y1="43.561" x2="52.451" y2="43.688" width="0.8128" layer="1"/>
 </signal>
 <signal name="SD_MISOV1">

Commit message: v2.1
Parts:
- added JP11, JP12, JP13: (no value), SparkFun:1X03
- added JP5, JP9: (no value), SparkFun:1X04_NO_SILK
- JP1: device SparkFun:1X04_NO_SILK -> SparkFun:1X03
- moved JP1 59.5 mm to (20.4, 9.02)
- moved JP8 51.5 mm to (67.0, 33.7), turned to 180 degrees
- moved SJ3 5.51 mm to (28.2, 56.4)
- moved JP7 4.87 mm to (31.4, 59.1)
Connections:
- new net 3V3: JP17.2, JP9.1
- new net N$1: D1.A, JP1.3, JP12.3
- new net N$2: JP1.1, JP12.1
- new net N$6: JP11.1, JP13.1
- new net N$7: JP11.2, JP13.2
- new net N$8: JP11.3, JP13.3
- net GND: now also JP5.1
- net N$3: now also JP1.2, JP12.2; no longer D1.A, JP8.3
- net SD_CD: now also JP5.4, JP8.2; no longer JP1.3
- net SD_CS: now also JP8.1, JP9.3; no longer JP1.4
- net SD_MISO: now also JP9.2
- net SD_MOSI: now also JP5.2
- net SD_SCK: now also JP5.3
Routing:
- net SD_CS: track 36.5 -> 68.7 mm, vias 1 -> 3
- net SD_MOSI: track 23.8 -> 54.9 mm, vias 0 -> 2
- net SD_SCK: track 23.7 -> 49.1 mm
- net 3V3: track 0.00 -> 25.0 mm
- net SD_CD: track 47.9 -> 69.7 mm
- net SD_MISO: track 32.3 -> 51.4 mm
- net GND: track 81.8 -> 100.5 mm, vias 0 -> 1
- net N$1: track 0.00 -> 9.08 mm
- net VBB: track 75.2 -> 83.3 mm
- net SD_MISOV1: track 21.3 -> 16.7 mm
- net N$3: track 6.40 -> 2.54 mm
- net N$8: track 0.00 -> 2.54 mm
- net N$7: track 0.00 -> 2.54 mm
- net N$6: track 0.00 -> 2.54 mm
- net N$2: track 0.00 -> 2.54 mm
Other:
- board size 62.9 x 67.9 mm -> 68.2 x 70.1 mm
- board text added: "EXT-SD"
- board text added: "by Laurent LE GOFF"
- board text added: "v2.1"
- board text removed: "3v3"
