File: SmoothieboardGlcdAdapter2.sch (EAGLE design)
At the start: 16 parts, among them IC1 7805TV

Commit message: v2.1
Parts:
- added JP11, JP12, JP13: (no value), SparkFun:M03PTH
- added JP5, JP9: (no value), SparkFun:M041X04_NO_SILK
- JP1: device SparkFun:M041X04_NO_SILK -> SparkFun:M03PTH
Connections:
- new net 3V3: JP17.2, JP9.1
- new net N$1: D1.A, JP1.3, JP12.3
- new net N$2: JP1.1, JP12.1
- new net N$6: JP11.1, JP13.1
- new net N$7: JP11.2, JP13.2
- new net N$8: JP11.3, JP13.3
- net GND: now also JP5.1
- net N$3: now also JP1.2, JP12.2; no longer D1.A, JP8.3
- net SD_CD: now also JP5.4, JP8.2; no longer JP1.3
- net SD_CS: now also JP8.1, JP9.3; no longer JP1.4
- net SD_MISO: now also JP9.2
- net SD_MOSI: now also JP5.2
- net SD_SCK: now also JP5.3
Other:
- note added: "by: Laurent LE GOFF"
- note removed: "by: Arthur Wolf"
- note removed: "produced by: Trinity Labs"
- moved on the sheet: JP8
